Commit message: added turtlebot3 common mesh

File: src/dtn_sim/urdf/turtlebot3_pi_dtn.urdf (robot description, URDF)
Before this commit: robot turtlebot3_dtn, 7 links, 6 joints
Links:
- added link base_scan, mass 0.114; collision cylinder length=0.0315 radius=0.055; visual mesh filename=package://dtn_sim/models/turtlebot3_common/meshes/lds.dae scale=0.001 0.001 0.001
- added link camera_link; collision box size=0.015 0.030 0.027
- added link camera_rgb_frame
- added link camera_rgb_optical_frame
- link base_link: geometry collision box size=0.266 0.266 0.094; visual mesh filename=package://dtn_sim/models/turtlebot3_common/meshes/waffle_pi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 scale=0.001 0.001 0.001
- link wheel_left_link: geometry collision cylinder length=0.018 radius=0.033; visual mesh filename=package://dtn_sim/models/turtlebot3_common/meshes/tire.dae scale=0.001 0.001 0.001
- link wheel_right_link: geometry collision cylinder length=0.018 radius=0.033; visual mesh filename=package://dtn_sim/models/turtlebot3_common/meshes/tire.dae scale=0.001 0.001 0.001
Joints:
- added joint camera_joint: type fixed, parent base_link, child camera_link, origin xyz=0.073 -0.011 0.084 rpy=0 0 0
- added joint camera_rgb_joint: type fixed, parent camera_link, child camera_rgb_frame, origin xyz=0.003 0.011 0.009 rpy=0 0 0
- added joint camera_rgb_optical_joint: type fixed, parent camera_rgb_frame, child camera_rgb_optical_frame, origin xyz=0 0 0 rpy=-1.57 0 -1.57
- added joint scan_joint: type fixed, parent base_link, child base_scan, origin xyz=-0.064 0 0.122 rpy=0 0 0

Commit message: finally got sim working

File: src/dtn_sim/urdf/turtlebot3_pi_dtn.urdf (robot description, URDF)
Before this commit: robot turtlebot3_dtn, 11 links, 10 joints
Links:
- removed link base_scan
- removed link camera_link
- removed link camera_rgb_frame
- removed link camera_rgb_optical_frame
Joints:
- removed joint camera_joint
- removed joint camera_rgb_joint
- removed joint camera_rgb_optical_joint
- removed joint scan_joint
